Commit message: Still doesnt work

File: arm_description/urdf/phantomx_reactor_wrist.urdf.xacro (robot description, xacro)
@@ -32,5 +32,5 @@
 			  <origin xyz="0 0 0" rpy="0 0 0" />
 			  <geometry>
-				<mesh filename="package://phantomx_reactor_arm_description/meshes/base_link.STL" />
+				<mesh filename="package://arm_description/meshes/base_link.STL" />
 			  </geometry>
 			  <material name="">
@@ -41,5 +41,5 @@
 			  <origin xyz="0 0 0" rpy="0 0 0" />
 			  <geometry>
-				<mesh filename="package://phantomx_reactor_arm_description/meshes/base_link_hull.STL" />
+				<mesh filename="package://arm_description/meshes/base_link_hull.STL" />
 			  </geometry>
 			</collision>
@@ -63,5 +63,5 @@
 			  <origin xyz="0 0 0" rpy="0 0 0" />
 			  <geometry>
-				<mesh   filename="package://phantomx_reactor_arm_description/meshes/shoulder_link.STL" />
+				<mesh   filename="package://arm_description/meshes/shoulder_link.STL" />
 			  </geometry>
 			  <material
@@ -73,5 +73,5 @@
 			  <origin xyz="0 0 0" rpy="0 0 0" />
 			  <geometry>
-				<mesh   filename="package://phantomx_reactor_arm_description/meshes/shoulder_link_hull.STL" />
+				<mesh   filename="package://arm_description/meshes/shoulder_link_hull.STL" />
 			  </geometry>
 			</collision>
@@ -96,5 +96,5 @@
 			  <origin xyz="0 0 0" rpy="-${PI/2} 0 -${PI/2}" />
 			  <geometry>
-				<mesh filename="package://phantomx_reactor_arm_description/meshes/bicep_link.STL" />
+				<mesh filename="package://arm_description/meshes/bicep_link.STL" />
 			  </geometry>
 			  <material name="">
@@ -105,5 +105,5 @@
 			  <origin xyz="0 0 0" rpy="-${PI/2} 0 -${PI/2}" />
 			  <geometry>
-				<mesh filename="package://phantomx_reactor_arm_description/meshes/bicep_link_hull.STL" />
+				<mesh filename="package://arm_description/meshes/bicep_link_hull.STL" />
 			  </geometry>
 			</collision>
@@ -127,14 +127,14 @@
 				<origin xyz="0 0 0" rpy="0 0 0" />
 				<geometry>
-					<mesh filename="package://phantomx_reactor_arm_description/meshes/forearm_link.STL" />
-				</geometry>
-				<material name="">
-					<color rgba="0.25098 0.25098 0.25098 1" />
-				</material>
-			</visual>
-			<collision>
-				<origin xyz="0 0 0" rpy="0 0 0" />
-				<geometry>
-					<mesh filename="package://phantomx_reactor_arm_description/meshes/forearm_link_hull.STL" />
+					<mesh filename="package://arm_description/meshes/forearm_link.STL" />
+				</geometry>
+				<material name="">
+					<color rgba="0.25098 0.25098 0.25098 1" />
+				</material>
+			</visual>
+			<collision>
+				<origin xyz="0 0 0" rpy="0 0 0" />
+				<geometry>
+					<mesh filename="package://arm_description/meshes/forearm_link_hull.STL" />
 				</geometry>
 			</collision>
@@ -159,14 +159,14 @@
 				<origin xyz="0 0 0" rpy="0 0 0" />
 				<geometry>
-					<mesh filename="package://phantomx_reactor_arm_description/meshes/wrist_1.STL" />
-				</geometry>
-				<material name="">
-					<color rgba="0.25098 0.25098 0.25098 1" />
-				</material>
-			</visual>
-			<collision>
-				<origin xyz="0 0 0" rpy="0 0 0" />
-				<geometry>
-					<mesh filename="package://phantomx_reactor_arm_description/meshes/wrist_1_hull.STL" />
+					<mesh filename="package://arm_description/meshes/wrist_1.STL" />
+				</geometry>
+				<material name="">
+					<color rgba="0.25098 0.25098 0.25098 1" />
+				</material>
+			</visual>
+			<collision>
+				<origin xyz="0 0 0" rpy="0 0 0" />
+				<geometry>
+					<mesh filename="package://arm_description/meshes/wrist_1_hull.STL" />
 				</geometry>
 			</collision>
@@ -191,14 +191,14 @@
 				<origin xyz="0 0 0" rpy="0 0 0" />
 				<geometry>
-					<mesh filename="package://phantomx_reactor_arm_description/meshes/wrist_2.STL" />
-				</geometry>
-				<material name="">
-					<color rgba="0.25098 0.25098 0.25098 1" />
-				</material>
-			</visual>
-			<collision>
-				<origin xyz="0 0 0" rpy="0 0 0" />
-				<geometry>
-					<mesh filename="package://phantomx_reactor_arm_description/meshes/wrist_2_hull.STL" />
+					<mesh filename="package://arm_description/meshes/wrist_2.STL" />
+				</geometry>
+				<material name="">
+					<color rgba="0.25098 0.25098 0.25098 1" />
+				</material>
+			</visual>
+			<collision>
+				<origin xyz="0 0 0" rpy="0 0 0" />
+				<geometry>
+					<mesh filename="package://arm_description/meshes/wrist_2_hull.STL" />
 				</geometry>
 			</collision>
@@ -221,5 +221,5 @@
 				<origin xyz="0 0 0" rpy="1.57 3.14 1.57" />
 				<geometry>
-					<mesh filename="package://phantomx_reactor_arm_description/meshes/Guide_Rail_Fixed_Centered.stl" scale="0.01 0.01 0.01" />
+					<mesh filename="package://arm_description/meshes/Guide_Rail_Fixed_Centered.stl" scale="0.01 0.01 0.01" />
 				</geometry>
 				<material name="">
@@ -230,5 +230,5 @@
 				<origin xyz="0 0 0" rpy="1.57 3.14 1.57" />
 				<geometry>
-					<mesh filename="package://phantomx_reactor_arm_description/meshes/Guide_Rail_Fixed_Centered.stl" scale="0.01 0.01 0.01" />
+					<mesh filename="package://arm_description/meshes/Guide_Rail_Fixed_Centered.stl" scale="0.01 0.01 0.01" />
 				</geometry>
 			</collision>
@@ -254,5 +254,5 @@
 				<origin xyz="0 0.010 0" rpy="-1.57 -1.57 0" />
 				<geometry>
-					<mesh filename="package://phantomx_reactor_arm_description/meshes/Gripper_Hand_Fixed_Centered.stl" scale="0.01 0.01 0.01" />
+					<mesh filename="package://arm_description/meshes/Gripper_Hand_Fixed_Centered.stl" scale="0.01 0.01 0.01" />
 				</geometry>
 				<material name="">
@@ -263,5 +263,5 @@
 				<origin xyz="0 0.010 0" rpy="-1.57 -1.57 0" />
 				<geometry>
-					<mesh filename="package://phantomx_reactor_arm_description/meshes/Gripper_Hand_Fixed_Centered.stl" scale="0.01 0.01 0.01" />
+					<mesh filename="package://arm_description/meshes/Gripper_Hand_Fixed_Centered.stl" scale="0.01 0.01 0.01" />
 				</geometry>
 			</collision>
@@ -279,5 +279,5 @@
 				<origin xyz="0 -0.010 0" rpy="1.57 1.57 0" />
 				<geometry>
-					<mesh filename="package://phantomx_reactor_arm_description/meshes/Gripper_Hand_Fixed_Centered.stl" scale="0.01 0.01 0.01" />
+					<mesh filename="package://arm_description/meshes/Gripper_Hand_Fixed_Centered.stl" scale="0.01 0.01 0.01" />
 				</geometry>
 				<material name="">
@@ -288,5 +288,5 @@
 				<origin xyz="0 -0.010 0" rpy="1.57 1.57 0" />
 				<geometry>
-					<mesh filename="package://phantomx_reactor_arm_description/meshes/Gripper_Hand_Fixed_Centered.stl" scale="0.01 0.01 0.01" />
+					<mesh filename="package://arm_description/meshes/Gripper_Hand_Fixed_Centered.stl" scale="0.01 0.01 0.01" />
 				</geometry>
 			</collision>

Commit message: IT LIVES

File: arm_description/urdf/phantomx_reactor_wrist.urdf.xacro (robot description, xacro)
@@ -9,5 +9,5 @@
 	<xacro:property name="elbow_pitch_joint_lower_limit" value="-2"/>
 	<xacro:property name="wrist_pitch_upper_limit" value="1.9"/>
-	<xacro:property name="wrist_pitch_lower_limit" value="-1.7"/>
+	<xacro:property name="wrist_pitch_lower_limit" value="-1.9"/>
 	<xacro:property name="wrist_roll_upper_limit" value="${PI}"/>
 	<xacro:property name="wrist_roll_lower_limit" value="-${PI}"/>
@@ -252,14 +252,14 @@
 		<link name="${prefix}gripper_right_link">
 			<visual>
-				<origin xyz="0 0.010 0" rpy="-1.57 -1.57 0" />
-				<geometry>
-					<mesh filename="package://arm_description/meshes/Gripper_Hand_Fixed_Centered.stl" scale="0.01 0.01 0.01" />
-				</geometry>
-				<material name="">
-					<color rgba="0.25098 0.25098 0.25098 1" />
-				</material>
-			</visual>
-			<collision>
-				<origin xyz="0 0.010 0" rpy="-1.57 -1.57 0" />
+				<origin xyz="0 0.0150 0" rpy="-1.57 -1.57 0" />
+				<geometry>
+					<mesh filename="package://arm_description/meshes/Gripper_Hand_Fixed_Centered.stl" scale="0.01 0.01 0.01" />
+				</geometry>
+				<material name="">
+					<color rgba="0.25098 0.25098 0.25098 1" />
+				</material>
+			</visual>
+			<collision>
+				<origin xyz="0 0.0150 0" rpy="-1.57 -1.57 0" />
 				<geometry>
 					<mesh filename="package://arm_description/meshes/Gripper_Hand_Fixed_Centered.stl" scale="0.01 0.01 0.01" />
@@ -277,14 +277,14 @@
 		<link name="${prefix}gripper_left_link">
 			<visual>
-				<origin xyz="0 -0.010 0" rpy="1.57 1.57 0" />
-				<geometry>
-					<mesh filename="package://arm_description/meshes/Gripper_Hand_Fixed_Centered.stl" scale="0.01 0.01 0.01" />
-				</geometry>
-				<material name="">
-					<color rgba="0.25098 0.25098 0.25098 1" />
-				</material>
-			</visual>
-			<collision>
-				<origin xyz="0 -0.010 0" rpy="1.57 1.57 0" />
+				<origin xyz="0 -0.0150 0" rpy="1.57 1.57 0" />
+				<geometry>
+					<mesh filename="package://arm_description/meshes/Gripper_Hand_Fixed_Centered.stl" scale="0.01 0.01 0.01" />
+				</geometry>
+				<material name="">
+					<color rgba="0.25098 0.25098 0.25098 1" />
+				</material>
+			</visual>
+			<collision>
+				<origin xyz="0 -0.0150 0" rpy="1.57 1.57 0" />
 				<geometry>
 					<mesh filename="package://arm_description/meshes/Gripper_Hand_Fixed_Centered.stl" scale="0.01 0.01 0.01" />

Commit message: working

File: arm_description/urdf/phantomx_reactor_wrist.urdf.xacro (robot description, xacro)
@@ -12,14 +12,14 @@
 	<xacro:property name="wrist_roll_upper_limit" value="${PI}"/>
 	<xacro:property name="wrist_roll_lower_limit" value="-${PI}"/>
-	<xacro:property name="gripper_joint_upper_limit" value="0.0"/>
-	<xacro:property name="gripper_joint_lower_limit" value="0.03"/>
+	<xacro:property name="gripper_joint_upper_limit" value="0.04"/>
+	<xacro:property name="gripper_joint_lower_limit" value="0.0"/>
 	<xacro:macro name="phantomx_reactor_wrist" params="parent prefix *origin">
-	    <!-- ARM BASE JOINT -->
+	  <!-- ARM BASE JOINT -->
 		<joint name="${prefix}base_joint" type="fixed">
 			<insert_block name="origin" />
 			<parent link="${parent}" />
-			<child link="${prefix}base_link" />
-		</joint>
-		<link name="${prefix}base_link">
+			<child link="arm_base_link" />
+		</joint>
+		<link name="arm_base_link">
 			<inertial>
 			  <origin xyz="-3.9657E-09 2.0144E-09 0.04262" rpy="0 0 0" />
@@ -49,5 +49,5 @@
 			<origin xyz="0 0 0.081" rpy="0 0 0" />
 			<!--origin xyz="0 0 0.081" rpy="0 0 0" /-->
-			<parent link="${prefix}base_link" />
+			<parent link="arm_base_link" />
 			<child link="${prefix}shoulder_link" />
 			<axis xyz="0 0 1" />
